Commit message: feat(ch13): integrate and verify MuJoCo model

File: Ch13/ros2_ws/src/integrated_robot_description/urdf/robot_system.urdf.xacro (robot description, xacro)
@@ -15,4 +15,20 @@
   <xacro:quadruped_base/>
   <xacro:manipulator_arm parent_link="base_link" prefix="arm_" xyz="0 0 0.095" rpy="0 0 0"/>
+  <joint name="lidar_mount_joint" type="fixed">
+    <parent link="base_link"/><child link="lidar_link"/><origin xyz="-0.18 0 0.12"/>
+  </joint>
+  <link name="lidar_link">
+    <visual><geometry><cylinder radius="0.035" length="0.045"/></geometry><material name="sensor_blue"/></visual>
+    <collision><geometry><cylinder radius="0.033" length="0.043"/></geometry></collision>
+    <xacro:cylinder_inertial mass="0.12" radius="0.035" length="0.045"/>
+  </link>
+  <joint name="camera_mount_joint" type="fixed">
+    <parent link="arm_link_6"/><child link="camera_link"/><origin xyz="0.03 0 0.03" rpy="0 -1.5708 0"/>
+  </joint>
+  <link name="camera_link">
+    <visual><geometry><box size="0.02 0.05 0.02"/></geometry><material name="body_black"/></visual>
+    <collision><geometry><box size="0.018 0.048 0.018"/></geometry></collision>
+    <xacro:box_inertial mass="0.05" x="0.02" y="0.05" z="0.02"/>
+  </link>
   <xacro:system_ros2_control name="IntegratedRobotSystem" backend="${backend}" mujoco_model_path="$(arg mujoco_model_path)"/>
   <xacro:if value="${backend == 'gazebo'}">

File: Ch13/ros2_ws/src/integrated_robot_description/urdf/system.ros2_control.xacro (robot description, xacro)
@@ -1,7 +1,7 @@
 <?xml version="1.0"?>
 <robot xmlns:xacro="http://www.ros.org/wiki/xacro">
-  <xacro:macro name="controlled_joint" params="name initial">
+  <xacro:macro name="controlled_joint" params="name initial lower upper">
     <joint name="${name}">
-      <command_interface name="position"><param name="min">-6.3</param><param name="max">6.3</param></command_interface>
+      <command_interface name="position"><param name="min">${lower}</param><param name="max">${upper}</param></command_interface>
       <state_interface name="position"><param name="initial_value">${initial}</param></state_interface>
       <state_interface name="velocity"/>
@@ -15,11 +15,11 @@
         <xacro:if value="${backend == 'mujoco'}"><plugin>mujoco_ros2_control/MujocoSystemInterface</plugin><param name="mujoco_model">${mujoco_model_path}</param></xacro:if>
       </hardware>
-      <xacro:controlled_joint name="fr_hip_joint" initial="0"/><xacro:controlled_joint name="fr_thigh_joint" initial="-0.5"/><xacro:controlled_joint name="fr_calf_joint" initial="1.0"/>
-      <xacro:controlled_joint name="fl_hip_joint" initial="0"/><xacro:controlled_joint name="fl_thigh_joint" initial="-0.5"/><xacro:controlled_joint name="fl_calf_joint" initial="1.0"/>
-      <xacro:controlled_joint name="rr_hip_joint" initial="0"/><xacro:controlled_joint name="rr_thigh_joint" initial="-0.5"/><xacro:controlled_joint name="rr_calf_joint" initial="1.0"/>
-      <xacro:controlled_joint name="rl_hip_joint" initial="0"/><xacro:controlled_joint name="rl_thigh_joint" initial="-0.5"/><xacro:controlled_joint name="rl_calf_joint" initial="1.0"/>
-      <xacro:controlled_joint name="arm_joint_1" initial="0"/><xacro:controlled_joint name="arm_joint_2" initial="0"/><xacro:controlled_joint name="arm_joint_3" initial="0"/>
-      <xacro:controlled_joint name="arm_joint_4" initial="0"/><xacro:controlled_joint name="arm_joint_5" initial="0"/><xacro:controlled_joint name="arm_joint_6" initial="0"/>
-      <xacro:controlled_joint name="gripper_left_joint" initial="0.015"/><xacro:controlled_joint name="gripper_right_joint" initial="0.015"/>
+      <xacro:controlled_joint name="fr_hip_joint" initial="0" lower="-0.8" upper="0.8"/><xacro:controlled_joint name="fr_thigh_joint" initial="-0.5" lower="-1.0" upper="4.0"/><xacro:controlled_joint name="fr_calf_joint" initial="1.0" lower="-2.8" upper="2.8"/>
+      <xacro:controlled_joint name="fl_hip_joint" initial="0" lower="-0.8" upper="0.8"/><xacro:controlled_joint name="fl_thigh_joint" initial="-0.5" lower="-1.0" upper="4.0"/><xacro:controlled_joint name="fl_calf_joint" initial="1.0" lower="-2.8" upper="2.8"/>
+      <xacro:controlled_joint name="rr_hip_joint" initial="0" lower="-0.8" upper="0.8"/><xacro:controlled_joint name="rr_thigh_joint" initial="-0.5" lower="-1.0" upper="4.0"/><xacro:controlled_joint name="rr_calf_joint" initial="1.0" lower="-2.8" upper="2.8"/>
+      <xacro:controlled_joint name="rl_hip_joint" initial="0" lower="-0.8" upper="0.8"/><xacro:controlled_joint name="rl_thigh_joint" initial="-0.5" lower="-1.0" upper="4.0"/><xacro:controlled_joint name="rl_calf_joint" initial="1.0" lower="-2.8" upper="2.8"/>
+      <xacro:controlled_joint name="arm_joint_1" initial="0" lower="-3.14159" upper="3.14159"/><xacro:controlled_joint name="arm_joint_2" initial="0" lower="-1.5708" upper="1.5708"/><xacro:controlled_joint name="arm_joint_3" initial="0" lower="-2.0944" upper="2.0944"/>
+      <xacro:controlled_joint name="arm_joint_4" initial="0" lower="-3.14159" upper="3.14159"/><xacro:controlled_joint name="arm_joint_5" initial="0" lower="-1.5708" upper="1.5708"/><xacro:controlled_joint name="arm_joint_6" initial="0" lower="-3.14159" upper="3.14159"/>
+      <xacro:controlled_joint name="gripper_left_joint" initial="0.015" lower="0" upper="0.03"/><xacro:controlled_joint name="gripper_right_joint" initial="0.015" lower="0" upper="0.03"/>
     </ros2_control>
   </xacro:macro>

Commit message: feat(ch13): add native eye-in-hand RGB-D and optical frames

File: Ch13/ros2_ws/src/integrated_robot_description/urdf/robot_system.urdf.xacro (robot description, xacro)
@@ -4,4 +4,5 @@
   <xacro:arg name="controllers_file" default="config/controllers.yaml"/>
   <xacro:arg name="mujoco_model_path" default="mujoco/robot_system.xml"/>
+  <xacro:arg name="vision_enabled" default="false"/>
   <xacro:include filename="materials.xacro"/>
   <xacro:include filename="inertial_macros.xacro"/>
@@ -9,4 +10,5 @@
   <xacro:include filename="manipulator.xacro"/>
   <xacro:include filename="system.ros2_control.xacro"/>
+  <xacro:include filename="vision_sensors.xacro"/>
   <xacro:property name="backend" value="$(arg control_backend)"/>
   <xacro:unless value="${backend in ['mock', 'gazebo', 'mujoco']}">
@@ -24,5 +26,5 @@
   </link>
   <joint name="camera_mount_joint" type="fixed">
-    <parent link="arm_link_6"/><child link="camera_link"/><origin xyz="0.03 0 0.03" rpy="0 -1.5708 0"/>
+    <parent link="arm_link_6"/><child link="camera_link"/><origin xyz="0.03 0 0.03" rpy="0 ${-pi/2} 0"/>
   </joint>
   <link name="camera_link">
@@ -31,4 +33,7 @@
     <xacro:box_inertial mass="0.05" x="0.02" y="0.05" z="0.02"/>
   </link>
+  <xacro:if value="$(arg vision_enabled)">
+    <xacro:vision_frames enabled="true"/>
+  </xacro:if>
   <xacro:system_ros2_control name="IntegratedRobotSystem" backend="${backend}" mujoco_model_path="$(arg mujoco_model_path)"/>
   <xacro:if value="${backend == 'gazebo'}">

Commit message: fix(ch13): diagnose vision latency and serialize tracking control ticks

File: Ch13/ros2_ws/src/integrated_robot_description/urdf/robot_system.urdf.xacro (robot description, xacro)
@@ -4,4 +4,5 @@
   <xacro:arg name="controllers_file" default="config/controllers.yaml"/>
   <xacro:arg name="mujoco_model_path" default="mujoco/robot_system.xml"/>
+  <xacro:arg name="mujoco_headless" default="false"/>
   <xacro:arg name="vision_enabled" default="false"/>
   <xacro:include filename="materials.xacro"/>
@@ -36,5 +37,5 @@
     <xacro:vision_frames enabled="true"/>
   </xacro:if>
-  <xacro:system_ros2_control name="IntegratedRobotSystem" backend="${backend}" mujoco_model_path="$(arg mujoco_model_path)"/>
+  <xacro:system_ros2_control name="IntegratedRobotSystem" backend="${backend}" mujoco_model_path="$(arg mujoco_model_path)" mujoco_headless="$(arg mujoco_headless)"/>
   <xacro:if value="${backend == 'gazebo'}">
     <gazebo>

File: Ch13/ros2_ws/src/integrated_robot_description/urdf/system.ros2_control.xacro (robot description, xacro)
@@ -8,10 +8,10 @@
     </joint>
   </xacro:macro>
-  <xacro:macro name="system_ros2_control" params="name backend mujoco_model_path">
+  <xacro:macro name="system_ros2_control" params="name backend mujoco_model_path mujoco_headless:=false">
     <ros2_control name="${name}" type="system">
       <hardware>
         <xacro:if value="${backend == 'mock'}"><plugin>mock_components/GenericSystem</plugin><param name="calculate_dynamics">false</param></xacro:if>
         <xacro:if value="${backend == 'gazebo'}"><plugin>gz_ros2_control/GazeboSimSystem</plugin></xacro:if>
-        <xacro:if value="${backend == 'mujoco'}"><plugin>mujoco_ros2_control/MujocoSystemInterface</plugin><param name="mujoco_model">${mujoco_model_path}</param></xacro:if>
+        <xacro:if value="${backend == 'mujoco'}"><plugin>mujoco_ros2_control/MujocoSystemInterface</plugin><param name="mujoco_model">${mujoco_model_path}</param><param name="headless">${str(mujoco_headless).lower()}</param></xacro:if>
       </hardware>
       <xacro:controlled_joint name="fr_hip_joint" initial="0" lower="-0.8" upper="0.8"/><xacro:controlled_joint name="fr_thigh_joint" initial="-0.5" lower="-1.0" upper="4.0"/><xacro:controlled_joint name="fr_calf_joint" initial="1.0" lower="-2.8" upper="2.8"/>

Commit message: fix(ch13): prevent duplicate legacy rendering with snapshot camera

File: Ch13/ros2_ws/src/integrated_robot_description/urdf/robot_system.urdf.xacro (robot description, xacro)
@@ -5,4 +5,5 @@
   <xacro:arg name="mujoco_model_path" default="mujoco/robot_system.xml"/>
   <xacro:arg name="mujoco_headless" default="false"/>
+  <xacro:arg name="mujoco_auto_register_cameras" default="true"/>
   <xacro:arg name="vision_enabled" default="false"/>
   <xacro:include filename="materials.xacro"/>
@@ -37,5 +38,5 @@
     <xacro:vision_frames enabled="true"/>
   </xacro:if>
-  <xacro:system_ros2_control name="IntegratedRobotSystem" backend="${backend}" mujoco_model_path="$(arg mujoco_model_path)" mujoco_headless="$(arg mujoco_headless)"/>
+  <xacro:system_ros2_control name="IntegratedRobotSystem" backend="${backend}" mujoco_model_path="$(arg mujoco_model_path)" mujoco_headless="$(arg mujoco_headless)" mujoco_auto_register_cameras="$(arg mujoco_auto_register_cameras)"/>
   <xacro:if value="${backend == 'gazebo'}">
     <gazebo>

File: Ch13/ros2_ws/src/integrated_robot_description/urdf/system.ros2_control.xacro (robot description, xacro)
@@ -8,10 +8,10 @@
     </joint>
   </xacro:macro>
-  <xacro:macro name="system_ros2_control" params="name backend mujoco_model_path mujoco_headless:=false">
+  <xacro:macro name="system_ros2_control" params="name backend mujoco_model_path mujoco_headless:=false mujoco_auto_register_cameras:=true">
     <ros2_control name="${name}" type="system">
       <hardware>
         <xacro:if value="${backend == 'mock'}"><plugin>mock_components/GenericSystem</plugin><param name="calculate_dynamics">false</param></xacro:if>
         <xacro:if value="${backend == 'gazebo'}"><plugin>gz_ros2_control/GazeboSimSystem</plugin></xacro:if>
-        <xacro:if value="${backend == 'mujoco'}"><plugin>mujoco_ros2_control/MujocoSystemInterface</plugin><param name="mujoco_model">${mujoco_model_path}</param><param name="headless">${str(mujoco_headless).lower()}</param></xacro:if>
+        <xacro:if value="${backend == 'mujoco'}"><plugin>mujoco_ros2_control/MujocoSystemInterface</plugin><param name="mujoco_model">${mujoco_model_path}</param><param name="headless">${str(mujoco_headless).lower()}</param><param name="auto_register_cameras">${str(mujoco_auto_register_cameras).lower()}</param></xacro:if>
       </hardware>
       <xacro:controlled_joint name="fr_hip_joint" initial="0" lower="-0.8" upper="0.8"/><xacro:controlled_joint name="fr_thigh_joint" initial="-0.5" lower="-1.0" upper="4.0"/><xacro:controlled_joint name="fr_calf_joint" initial="1.0" lower="-2.8" upper="2.8"/>
