Commit message: fix(ch03): align link collision shapes and box inertia with visuals

File: Ch03/ros2_ws/src/my_robot_description/urdf/two_dof_arm.urdf (robot description, URDF)
Before this commit: robot two_dof_arm, 4 links, 3 joints
Links:
- link link1: geometry collision box size=0.05 0.05 0.5; visual box size=0.05 0.05 0.5
