Commit message: fix(ch03-3.3): correct Xacro inertia axes COM and EE chain

File: Ch03/ros2_ws/src/my_robot_description/urdf/two_dof_arm.urdf.xacro (robot description, xacro)
@@ -8,12 +8,14 @@
   <xacro:macro name="box_inertia" params="m w h d">
     <inertial>
+      <origin xyz="0 0 ${h/2}" rpy="0 0 0"/>
       <mass value="${m}"/>
       <inertia ixx="${(m/12) * (h*h + d*d)}" ixy="0.0" ixz="0.0"
-               iyy="${(m/12) * (w*w + d*d)}" iyz="0.0"
-               izz="${(m/12) * (w*w + h*h)}"/>
+               iyy="${(m/12) * (w*w + h*h)}" iyz="0.0"
+               izz="${(m/12) * (w*w + d*d)}"/>
     </inertial>
   </xacro:macro>
   <xacro:macro name="cylinder_inertia" params="m r h">
     <inertial>
+      <origin xyz="0 0 ${h/2}" rpy="0 0 0"/>
       <mass value="${m}"/>
       <inertia ixx="${(m/12) * (3*r*r + h*h)}" ixy="0.0" ixz="0.0"
@@ -79,4 +81,20 @@
     <limit lower="-1.57" upper="1.57" effort="100" velocity="1.0"/>
   </joint>
+  <!-- 3.2 정적 URDF와 TF 체인을 일치시키는 고정 말단 좌표계 -->
+  <joint name="joint_ee" type="fixed">
+    <parent link="link2"/>
+    <child link="end_effector_link"/>
+    <origin xyz="0 0 ${link_len}" rpy="0 0 0"/>
+  </joint>
+  <link name="end_effector_link">
+    <visual><geometry><sphere radius="0.02"/></geometry>
+      <material name="red"><color rgba="1 0 0 1"/></material>
+    </visual>
+    <collision><geometry><sphere radius="0.02"/></geometry></collision>
+    <inertial>
+      <mass value="0.01"/>
+      <inertia ixx="0.0000016" ixy="0" ixz="0" iyy="0.0000016" iyz="0" izz="0.0000016"/>
+    </inertial>
+  </link>
   <gazebo>
     <plugin filename="gz-sim-joint-state-publisher-system"

Commit message: fix(ch03): bound joint1 controller command and align dynamics settings

File: Ch03/ros2_ws/src/my_robot_description/urdf/two_dof_arm.urdf.xacro (robot description, xacro)
@@ -70,4 +70,5 @@
     <axis xyz="0 0 1"/>
     <limit lower="-3.14" upper="3.14" effort="100" velocity="1.0"/>
+    <dynamics damping="0.1" friction="0.05"/>
   </joint>
   <xacro:arm_link_macro name="link2" color_name="yellow" r="1" g="1" b="0"/>
@@ -78,4 +79,5 @@
     <axis xyz="0 1 0"/>
     <limit lower="-1.57" upper="1.57" effort="100" velocity="1.0"/>
+    <dynamics damping="0.1" friction="0.05"/>
   </joint>
   <gazebo>
@@ -96,6 +98,6 @@
       <i_max>1</i_max>
       <i_min>-1</i_min>
-      <cmd_max>1000</cmd_max>
-      <cmd_min>-1000</cmd_min>
+      <cmd_max>100</cmd_max>
+      <cmd_min>-100</cmd_min>
       <initial_position>0.0</initial_position>
     </plugin>
