Commit message: fix(ch09.1): correct model / launch contracts; document static checks

File: Ch09/ros2_ws/src/my_quadruped_bot/urdf/parts/leg.xacro (robot description, xacro)
@@ -11,13 +11,14 @@
     <link name="${prefix}_hip_link">
       <visual>
-        <origin xyz="0 0 0" rpy="0 0 0"/>
-        <geometry><box size="${hip_length} 0.04 0.04"/></geometry>
+        <origin xyz="0 ${y_reflect * hip_length / 2.0} 0" rpy="0 0 0"/>
+        <geometry><box size="0.04 ${hip_length} 0.04"/></geometry>
         <material name="grey"/>
       </visual>
       <collision>
-        <origin xyz="0 0 0" rpy="0 0 0"/>
-        <geometry><box size="${hip_length} 0.04 0.04"/></geometry>
+        <origin xyz="0 ${y_reflect * hip_length / 2.0} 0" rpy="0 0 0"/>
+        <geometry><box size="0.04 ${hip_length} 0.04"/></geometry>
       </collision>
-      <xacro:box_inertia m="${hip_mass}" x="${hip_length}" y="0.04" z="0.04" xyz="0 0 0" rpy="0 0 0"/>
+      <!-- Hip is a lateral bar along +Y/-Y, not the body X axis. -->
+      <xacro:box_inertia m="${hip_mass}" x="0.04" y="${hip_length}" z="0.04" xyz="0 ${y_reflect * hip_length / 2.0} 0" rpy="0 0 0"/>
     </link>
     <joint name="${prefix}_thigh_joint" type="revolute">

Commit message: revert(ch09.1): defer code changes until documentation PR is merged
Restore exact docs-only tree; saved complete code/test revisions in hold/ch09-section-9-1-code-fixes-20261021. No force push.

File: Ch09/ros2_ws/src/my_quadruped_bot/urdf/parts/leg.xacro (robot description, xacro)
@@ -11,14 +11,13 @@
     <link name="${prefix}_hip_link">
       <visual>
-        <origin xyz="0 ${y_reflect * hip_length / 2.0} 0" rpy="0 0 0"/>
-        <geometry><box size="0.04 ${hip_length} 0.04"/></geometry>
+        <origin xyz="0 0 0" rpy="0 0 0"/>
+        <geometry><box size="${hip_length} 0.04 0.04"/></geometry>
         <material name="grey"/>
       </visual>
       <collision>
-        <origin xyz="0 ${y_reflect * hip_length / 2.0} 0" rpy="0 0 0"/>
-        <geometry><box size="0.04 ${hip_length} 0.04"/></geometry>
+        <origin xyz="0 0 0" rpy="0 0 0"/>
+        <geometry><box size="${hip_length} 0.04 0.04"/></geometry>
       </collision>
-      <!-- Hip is a lateral bar along +Y/-Y, not the body X axis. -->
-      <xacro:box_inertia m="${hip_mass}" x="0.04" y="${hip_length}" z="0.04" xyz="0 ${y_reflect * hip_length / 2.0} 0" rpy="0 0 0"/>
+      <xacro:box_inertia m="${hip_mass}" x="${hip_length}" y="0.04" z="0.04" xyz="0 0 0" rpy="0 0 0"/>
     </link>
     <joint name="${prefix}_thigh_joint" type="revolute">
